File: FarmSupply.kicad_pcb (KiCad board)
At the start: 2 copper layers, 50.8 x 20.3 mm, 12 parts, among them P1 USB_C_Plug, P2 USB_C_Plug, P3 USB_C_Plug, P4 USB_C_Plug, P5 USB_C_Plug, P6 USB_C_Plug

Commit message: Add files via upload
Parts:
- added R10: 5.1k, Resistor_SMD:R_0805_2012Metric, F.Cu at (108.7, 90.2)
- added R11: 5.1k, Resistor_SMD:R_0805_2012Metric, F.Cu at (112.5, 90.2)
- added R12: 5.1k, Resistor_SMD:R_0805_2012Metric, F.Cu at (116.2, 90.2)
- added R13: 5.1k, Resistor_SMD:R_0805_2012Metric, B.Cu at (112.0, 83.2)
- added R2: 5.1k, Resistor_SMD:R_0805_2012Metric, F.Cu at (93.1, 90.2)
- added R3: 5.1k, Resistor_SMD:R_0805_2012Metric, B.Cu at (89.2, 97.2)
- added R4: 5.1k, Resistor_SMD:R_0805_2012Metric, F.Cu at (104.8, 90.2)
- added R5: 5.1k, Resistor_SMD:R_0805_2012Metric, F.Cu at (101.0, 90.2)
- added R6: 5.1k, Resistor_SMD:R_0805_2012Metric, F.Cu at (97.2, 90.2)
- added R7: 5.1k, Resistor_SMD:R_0805_2012Metric, B.Cu at (100.6, 96.5)
- added R8: 5.1k, Resistor_SMD:R_0805_2012Metric, F.Cu at (89.3, 90.2)
- added R9: 5.1k, Resistor_SMD:R_0805_2012Metric, F.Cu at (85.4, 90.2)
- P1, P2, P3, P4, P5, P6: value USB_C_Plug -> USB_C_Receptacle
- moved P3 12.7 mm to (111.8, 96.5), turned to 0 degrees
- moved P5 12.7 mm to (100.3, 83.8), turned to 180 degrees
- moved P4 11.7 mm to (111.8, 83.8)
- moved P2 10.8 mm to (100.3, 96.5)
- moved P6 0.05 mm to (88.9, 83.8)
Connections:
- P1 pad A5: unconnected-(P1-PadA5) -> Net-(P1-PadA5)
- P1 pad B5: unconnected-(P1-PadB5) -> Net-(P1-PadB5)
- P1 pad B6: (no net) -> unconnected-(P1-PadB6)
- P1 pad B7: (no net) -> unconnected-(P1-PadB7)
- P2 pad A5: unconnected-(P2-PadA5) -> Net-(P2-PadA5)
- P2 pad B5: unconnected-(P2-PadB5) -> Net-(P2-PadB5)
- P2 pad B6: (no net) -> unconnected-(P2-PadB6)
- P2 pad B7: (no net) -> unconnected-(P2-PadB7)
- P3 pad A5: unconnected-(P3-PadA5) -> Net-(P3-PadA5)
- P3 pad B5: unconnected-(P3-PadB5) -> Net-(P3-PadB5)
- P3 pad B6: (no net) -> unconnected-(P3-PadB6)
- P3 pad B7: (no net) -> unconnected-(P3-PadB7)
- P4 pad A5: unconnected-(P4-PadA5) -> Net-(P4-PadA5)
- P4 pad B5: unconnected-(P4-PadB5) -> Net-(P4-PadB5)
- P4 pad B6: (no net) -> unconnected-(P4-PadB6)
- P4 pad B7: (no net) -> unconnected-(P4-PadB7)
- P5 pad A5: unconnected-(P5-PadA5) -> Net-(P5-PadA5)
- P5 pad B5: unconnected-(P5-PadB5) -> Net-(P5-PadB5)
- P5 pad B6: (no net) -> unconnected-(P5-PadB6)
- P5 pad B7: (no net) -> unconnected-(P5-PadB7)
- P6 pad A5: unconnected-(P6-PadA5) -> Net-(P6-PadA5)
- P6 pad B5: unconnected-(P6-PadB5) -> Net-(P6-PadB5)
- P6 pad B6: (no net) -> unconnected-(P6-PadB6)
- P6 pad B7: (no net) -> unconnected-(P6-PadB7)
Routing:
- net GND: track 22.8 -> 42.0 mm, vias 0 -> 5
- net Net-(P1-PadA5): track 0.00 -> 6.53 mm
- net Net-(P1-PadB5): track 0.00 -> 5.04 mm, vias 0 -> 1
- net Net-(P4-PadB5): track 0.00 -> 4.62 mm, vias 0 -> 1
- net Net-(P2-PadB5): track 0.00 -> 4.40 mm, vias 0 -> 1
- net Net-(P4-PadA5): track 0.00 -> 4.31 mm
- net Net-(P5-PadA5): track 0.00 -> 4.31 mm
- net Net-(P5-PadB5): track 0.00 -> 3.81 mm
- net Net-(P2-PadA5): track 0.00 -> 3.62 mm
- net Net-(P3-PadA5): track 0.00 -> 3.59 mm
- net Net-(P6-PadB5): track 0.00 -> 3.58 mm
- net Net-(P6-PadA5): track 0.00 -> 3.26 mm
- net Net-(P3-PadB5): track 0.00 -> 3.25 mm
- net +5V: track 104.7 -> 104.1 mm
Other:
- board text removed: "USB IN"
